File: Seguidor de linea/pcb/eagle/ProyectoFinal.sch (EAGLE design)
At the start: 11 parts, among them IC1 MC9S08QE16CLD, IC2 L293D

Commit message: v1.0
Parts:
- removed BMX055: (no value), pinhead:PINHD-1X10
- removed LIPO7V: BATTERY 7V4, battery:AB9V
- removed PROGRAMADOR: (no value), pinhead:PINHD-1X3
- removed S1: (no value), switch-omron:10-XX
- removed U$1: WIRELESS-BLUETOOTH-HC-05, diy-modules:WIRELESS-BLUETOOTH-HC-05
- added 3V3, BKGD, GND: (no value), pinhead:PINHD-1X1
- added BLUETOOTH: hc-05, diy-modules:WIRELESS-BLUETOOTH-HC-05
- added BTN_START: (no value), switch-omron:10-XX
- added C1, C2, C4, C5: 0.1uF, rcl:C-EUC0805K
- added C7: 10uF, rcl:C-EUC1206K
- added CJMCU: (no value), pinhead:PINHD-1X4
- added LIPO, MOD3.3V, MOD3.3V1, MOD5V, MOD5V1: (no value), pinhead:PINHD-1X2
- added QTR8: (no value), pinhead:PINHD-1X11
Connections:
- removed net CSB1: BMX055.8
- removed net CSB2: BMX055.9
- removed net CSB3: BMX055.10
- removed net N$21: IC1.PTB3/KBI1P7/MOSI/ADP7, JP1.21
- removed net N$22: IC1.PTB2/KBI1P6/SPSCK/ADP6, JP1.22
- removed net N$23: IC1.PTB1/KBI1P5/TXD1/ADP5, JP2.1
- removed net N$24: IC1.PTB0/KBI1P4/RXD1/ADP4, JP2.2
- removed net N$26: IC1.PTA6/TPM1CH2/ADP8, JP2.4
- removed net N$27: IC1.VDD, JP2.5
- removed net N$28: IC1.VSS, JP2.6
- removed net N$32: IC1.PTA3/KBI1P3/SCL/ADP3, JP2.10
- removed net N$33: IC1.PTA2/KBI1P2/SDA/ADP2, JP2.11
- removed net N$4: LIPO7V.+, S1.P
- removed net N$5: IC1.VDDAD, JP1.5
- removed net N$6: IC1.VREFH, JP1.6
- removed net N$7: IC1.VREFL, JP1.7
- removed net N$8: IC1.VSSAD, JP1.8
- removed net PS: BMX055.5
- removed net SDO1: BMX055.6
- removed net SDO2: BMX055.7
- new net ADC2: IC1.PTA2/KBI1P2/SDA/ADP2, JP2.11, QTR8.3
- new net ADC3: IC1.PTA3/KBI1P3/SCL/ADP3, JP2.10, QTR8.4
- new net ADC4: IC1.PTB0/KBI1P4/RXD1/ADP4, JP2.2, QTR8.5
- new net ADC5: IC1.PTB1/KBI1P5/TXD1/ADP5, JP2.1, QTR8.6
- new net ADC6: IC1.PTB2/KBI1P6/SPSCK/ADP6, JP1.22, QTR8.7
- new net ADC7: IC1.PTB3/KBI1P7/MOSI/ADP7, JP1.21, QTR8.8
- new net ADC8: IC1.PTA6/TPM1CH2/ADP8, JP2.4, QTR8.9
- new net ADC9: QTR8.10
- new net R1: QTR8.2
- net 3V3: now also 3V3.1, C2.1, C5.2, C7.2, CJMCU.1, IC1.VDDAD, IC1.VREFH, JP1.5, JP1.6, MOD3.3V.1, MOD3.3V1.1; no longer BMX055.1, PROGRAMADOR.3
- net 5V: now also BLUETOOTH.+5V, C4.2, MOD5V.1, MOD5V1.1, QTR8.11; no longer U$1.+5V
- net 7V4: now also LIPO.1
- net BKGD: now also BKGD.1; no longer PROGRAMADOR.1
- net BTN_START: now also BTN_START.S, C1.2
- net GND: now also BLUETOOTH.GND, BTN_START.P, C1.1, C2.2, C4.1, C5.1, C7.1, CJMCU.2, GND.1, IC1.VREFL, IC1.VSS, IC1.VSSAD, JP1.7, JP1.8, JP2.6, LIPO.2, MOD3.3V.2, MOD3.3V1.2, MOD5V.2, MOD5V1.2, QTR8.1; no longer BMX055.2, LIPO7V.-, PROGRAMADOR.2, U$1.GND
- net RX_BT: now also BLUETOOTH.RX; no longer U$1.RX
- net SCL: now also CJMCU.3; no longer BMX055.3
- net SDA: now also CJMCU.4; no longer BMX055.4
- net TX_BT: now also BLUETOOTH.TX; no longer U$1.TX
Other:
- note added: "Módulo BlueTooth"
